File: PCB/PS_motherboard/hx711.kicad_sch (KiCad schematic)
At the start: 16 parts, among them U1 HX711

Commit message: Updated LCSC part numbers and footprints for all parts EXCEPT PB and Screw Terminals (added comments why not)
Parts:
- C1: footprint Capacitor_SMD:C_0603_1608Metric -> Capacitor_SMD:C_0402_1005Metric; Extended (none) -> 0; LCSC (none) -> C1525
- C2, C6: Extended (none) -> 0; LCSC (none) -> C19702
- C3, C4, C5, C7: Extended (none) -> 0; LCSC (none) -> C1525
- L1: footprint Inductor_SMD:L_0603_1608Metric -> (none)
- R3, R4: footprint Resistor_SMD:R_0402_1005Metric -> Resistor_SMD:R_0603_1608Metric; Extended (none) -> 0; LCSC (none) -> C22775
- R5: footprint Resistor_SMD:R_0402_1005Metric -> Resistor_SMD:R_0603_1608Metric; Extended (none) -> 0; LCSC (none) -> C22790
- R6: footprint Resistor_SMD:R_0402_1005Metric -> Resistor_SMD:R_0603_1608Metric; Extended (none) -> 0; LCSC (none) -> C22967
- R7: Extended (none) -> 0; LCSC (none) -> C25804
- U1: Extended (none) -> 1; LCSC (none) -> C6705483
- gave numbers to parts that had none: 1
Other:
- note added: "Mistake on the 8550 footprint Ryan: It looks correct (SOT-23) - will need to check with Montso"
- note removed: "Mistake on the 8550 footprint"

Commit message: Update footprints
Parts:
- L1: footprint (none) -> Inductor_SMD:L_0603_1608Metric; Extended (none) -> 1; LCSC (none) -> C275346
Changed lines of the file:
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@@
 			)
 		)
-		(property "Footprint" ""
+		(property "Footprint" "Inductor_SMD:L_0603_1608Metric"
 			(at 115.824 74.422 0)
 			(effects
@@
 			)
 		)
-		(property "Datasheet" "~"
+		(property "Datasheet" "https://wmsc.lcsc.com/wmsc/upload/file/pdf/v2/lcsc/2304140030_TDK-MLF1608A3R3JT000_C275346.pdf"
 			(at 115.824 74.422 0)
 			(effects
@@
 			(at 115.824 74.422 0)
 			(effects
+				(font
+					(size 1.27 1.27)
+				)
+				(hide yes)
+			)
+		)
+		(property "Extended" "1"
+			(at 115.824 74.422 0)
+			(effects
+				(font
+					(size 1.27 1.27)
+				)
+				(hide yes)
+			)
+		)
+		(property "LCSC" "C275346"
+			(at 115.824 74.422 0)
+			(effects
