File: PCB/PS_scale_v0/PS_scale_v0.kicad_sch (KiCad schematic)
At the start: 10 parts, among them J1 Screw_Terminal_01x04, J2 Conn_01x06_Socket, J3 Conn_01x04_Socket, J4 Conn_01x04_Socket, J5 Conn_01x05_Pin, J6 ESP32 DEVKIT

Commit message: Controller: Updated menu to have disconnect functionality.
Parts:
- removed J4: Conn_01x04_Socket, Connector_PinHeader_2.54mm:PinHeader_1x04_P2.54mm_Vertical, symbol Connector:Conn_01x04_Socket
- added BT1: CR2032, symbol Device:Battery_Cell
- added C1: 1uF, symbol Device:C_Small
- added C2: 100nF, symbol Device:C_Small
- added D1: 1N4148, Diode_THT:D_DO-35_SOD27_P7.62mm_Horizontal, symbol Diode:1N4148
- added J1: Screw_Terminal_01x06, TerminalBlock_Phoenix:TerminalBlock_Phoenix_PT-1,5-6-3.5-H_1x06_P3.50mm_Horizontal, symbol Connector:Screw_Terminal_01x06
- added J10: Micro_SD_Card, symbol Connector:Micro_SD_Card
- added J11: Conn_01x06_Pin, symbol Connector:Conn_01x06_Pin
- added J4: Conn_01x03_Socket, symbol Connector:Conn_01x03_Socket
- added J6: Conn_01x06_Socket, symbol Connector:Conn_01x06_Socket
- added J7: Conn_01x04_Socket, Connector_PinHeader_2.54mm:PinHeader_1x04_P2.54mm_Vertical, symbol Connector:Conn_01x04_Socket
- added JP1: Bat_Charge, symbol Jumper:SolderJumper_2_Open
- added JP2: 32kHz, symbol Jumper:SolderJumper_2_Open
- added R1, R2, R3, R5, R6, R7, R8: 4k7, symbol Device:R_Small_US
- added R4: 220R, symbol Device:R_Small_US
- added SW1: SW_Push, Button_Switch_SMD:SW_Push_1P1T_XKB_TS-1187A, symbol Switch:SW_Push
- added U1: DS3231M, Package_SO:SOIC-16W_7.5x10.3mm_P1.27mm, symbol Timer_RTC:DS3231M
- added U2: AT24CS32D-SSHM-T, Package_DFN_QFN:DFN-8-1EP_3x2mm_P0.5mm_EP1.3x1.5mm, symbol Memory_EEPROM:AT24CS32-MAHM
- renumbered D1 to D2, D2 to D3, J1 to J2, J2 to J3, J3 to J5, J5 to J8, J6 to J9, R2 to R10, R1 to R9
Connections:
- net E- is gone; now on net GND: J2.2 (Pin_2), J3.2 (Pin_2)
- net +3V3: now also C1.1, C2.1, J6.5 (Pin_5), J7.2 (Pin_2), JP1.1 (A), R1.1, R2.1, R3.1, R5.1, R6.1, R7.1, R8.1, SW1.2, U1.2 (VCC), U1.4 (~{RST}), U2.8 (VCC)
- net GND: now also BT1.2 (-), C1.2, C2.2, J1.2 (Pin_2), J11.6 (Pin_6), J7.1 (Pin_1), SW1.1, U1.10 (GND), U1.11 (GND), U1.12 (GND), U1.13 (GND), U1.5 (GND), U1.6 (GND), U1.7 (GND), U1.8 (GND), U1.9 (GND), U2.4 (GND), U2.7 (WP)
- net SCL: now also J6.1 (Pin_1), J7.3 (Pin_3), R5.2, U1.16 (SCL), U2.6 (SCL)
- net SDA: now also J6.2 (Pin_2), J7.4 (Pin_4), R6.2, U1.15 (SDA), U2.5 (SDA)
- net A+ renamed INA+
- net INA+: now also J1.4 (Pin_4)
- net A- renamed INA-
- net INA-: now also J1.3 (Pin_3)
- net E+ renamed EXC+
- net EXC+: now also J1.1 (Pin_1)
- new net: D1.2 (A), R4.2
- new net: JP2.2 (B), R7.2
- new net: JP1.2 (B), R4.1
- new net 32kHz: J6.3 (Pin_3), JP2.1 (A), U1.1 (32KHZ)
- new net A0: J4.1 (Pin_1), R3.2, U2.1 (A0)
- new net A1: J4.2 (Pin_2), R2.2, U2.2 (A1)
- new net A2: J4.3 (Pin_3), R1.2, U2.3 (A2)
- new net INB+: J1.6 (Pin_6)
- new net INB-: J1.5 (Pin_5)
- new net SD_CS: J11.1 (Pin_1)
- new net SD_MISO: J11.4 (Pin_4)
- new net SD_MOSI: J11.3 (Pin_3)
- new net SD_SCK: J11.2 (Pin_2)
- new net SD_VCC: J11.5 (Pin_5)
- new net SQW: J6.4 (Pin_4), R8.2, U1.3 (~{INT}/SQW)
- new net VDD: BT1.1 (+), D1.1 (K), J6.6 (Pin_6), U1.14 (VBAT)
- no-connect marks 3 -> 4
Other:
- added sheet HX711 (hx711.kicad_sch)
- note added: "HX711"
- note added: "No 1x6 Screw Terminals available on JLC"
- note added: "RST needs a pin on ESP"
